Commit message: bot model added

File: xacro/bot.xacro (robot description, xacro)
@@ -1,3 +1,57 @@
 <?xml version="1.0"?>
 <robot xmlns:xacro="http://www.ros.org/wiki/xacro" name="warehouse_robot">
+  <xacro:property name="PI" value="3.142" />
+  <xacro:macro name="wheel">
+    <inertial>
+      <origin xyz="1.404E-12 -1.4273E-06 -3.24719999991261E-12" rpy="0 0 0" />
+      <mass value="0.13417" />
+      <inertia ixx="0.000146905644650745" ixy="5.24655439786608E-15" ixz="1.58665244652452E-14" iyy="0.000279392456161737" iyz="-8.08703217025071E-15" izz="0.00014690564464536" />
+    </inertial>
+    <visual>
+      <origin xyz="0 0 0" rpy="0 0 0" />
+      <geometry>
+        <mesh filename="package://warehouse_robot/meshes/wheel.stl" />
+      </geometry>
+      <material name="">
+        <color rgba="0.79216 0.81961 0.93333 1" />
+      </material>
+    </visual>
+    <collision>
+      <origin xyz="0 0 0" rpy="1.5707963267949 0 0" />
+      <geometry>
+        <mesh filename="package://warehouse_robot/meshes/wheel.stl" />
+      </geometry>
+    </collision>
+  </xacro:macro>
+  <link name="base_link">
+  <inertial>
+    <origin xyz="0.089651 0.014045 0.000106459999999999" rpy="0 0 0" />
+    <mass value="4.9511" />
+    <inertia ixx="0.144771700464571" ixy="-0.00641450872692838" ixz="-0.00058647494980373" iyy="0.232027279470688" iyz="-0.000146713403145161" izz="0.369859293842831" />
+  </inertial>
+  <visual>
+    <origin xyz="0 0 0" rpy="${PI/2} 0 0" />
+    <geometry>
+      <mesh filename="package://warehouse_robot/meshes/bot.stl" />
+    </geometry>
+    <material name="">
+      <color rgba="0.79216 0.81961 0.93333 0.1" />
+    </material>
+  </visual>
+  <collision>
+    <origin xyz="0 0 0" rpy="0 0 0" />
+    <geometry>
+      <mesh filename="package://warehouse_robot/meshes/bot.stl" />
+    </geometry>
+  </collision>
+  </link>
+  <link name="wheel_1">
+  <xacro:wheel/>
+  </link>
+  <joint name="base_link_1" type="continuous">
+    <origin xyz="0 0 0" rpy="${PI/2} 0 0" />
+    <axis xyz="1 0 0" />
+    <parent link="base_link" />
+    <child link="wheel_1" />
+  </joint>
 </robot>

Commit message: added wheels

File: xacro/bot.xacro (robot description, xacro)
@@ -36,5 +36,5 @@
     </geometry>
     <material name="">
-      <color rgba="0.79216 0.81961 0.93333 0.1" />
+      <color rgba="0.79216 0.81961 0.93333 1" />
     </material>
   </visual>
@@ -46,12 +46,77 @@
   </collision>
   </link>
+  <!-- ===================== LEFT Wheels ============================= -->
   <link name="wheel_1">
   <xacro:wheel/>
   </link>
   <joint name="base_link_1" type="continuous">
-    <origin xyz="0 0 0" rpy="${PI/2} 0 0" />
+    <origin xyz="-0.26933 0.212 0" rpy="${PI/2} 0 0" />
     <axis xyz="1 0 0" />
     <parent link="base_link" />
     <child link="wheel_1" />
   </joint>
+  <link name="wheel_2">
+  <xacro:wheel/>
+  </link>
+  <joint name="base_link_2" type="continuous">
+    <origin xyz="-0.08 0.212 0" rpy="${PI/2} 0 0" />
+    <axis xyz="1 0 0" />
+    <parent link="base_link" />
+    <child link="wheel_2" />
+  </joint>
+  <link name="wheel_3">
+  <xacro:wheel/>
+  </link>
+  <joint name="base_link_3" type="continuous">
+    <origin xyz="0.10934 0.212 0" rpy="${PI/2} 0 0" />
+    <axis xyz="1 0 0" />
+    <parent link="base_link" />
+    <child link="wheel_3" />
+  </joint>
+  <link name="wheel_4">
+  <xacro:wheel/>
+  </link>
+  <joint name="base_link_4" type="continuous">
+    <origin xyz="0.29867 0.212 0" rpy="${PI/2} 0 0" />
+    <axis xyz="1 0 0" />
+    <parent link="base_link" />
+    <child link="wheel_4" />
+  </joint>
+  <!-- ===================== RIGHT Wheels ============================= -->
+  <link name="wheel_5">
+  <xacro:wheel/>
+  </link>
+  <joint name="base_link_5" type="continuous">
+    <origin xyz="-0.26933 -0.212 0" rpy="${PI/2} 0 0" />
+    <axis xyz="1 0 0" />
+    <parent link="base_link" />
+    <child link="wheel_5" />
+  </joint>
+  <link name="wheel_6">
+  <xacro:wheel/>
+  </link>
+  <joint name="base_link_6" type="continuous">
+    <origin xyz="-0.08 -0.212 0" rpy="${PI/2} 0 0" />
+    <axis xyz="1 0 0" />
+    <parent link="base_link" />
+    <child link="wheel_6" />
+  </joint>
+  <link name="wheel_7">
+  <xacro:wheel/>
+  </link>
+  <joint name="base_link_7" type="continuous">
+    <origin xyz="0.10934 -0.212 0" rpy="${PI/2} 0 0" />
+    <axis xyz="1 0 0" />
+    <parent link="base_link" />
+    <child link="wheel_7" />
+  </joint>
+  <link name="wheel_8">
+  <xacro:wheel/>
+  </link>
+  <joint name="base_link_8" type="continuous">
+    <origin xyz="0.29867 -0.212 0" rpy="${PI/2} 0 0" />
+    <axis xyz="1 0 0" />
+    <parent link="base_link" />
+    <child link="wheel_8" />
+  </joint>
 </robot>

Commit message: updated axes of wheels

File: xacro/bot.xacro (robot description, xacro)
@@ -51,6 +51,6 @@
   </link>
   <joint name="base_link_1" type="continuous">
-    <origin xyz="-0.26933 0.212 0" rpy="${PI/2} 0 0" />
-    <axis xyz="1 0 0" />
+    <origin xyz="-0.26933 0.212 0" rpy="-${PI/2} -${PI/2} 0" />
+    <axis xyz="0 0 1" />
     <parent link="base_link" />
     <child link="wheel_1" />
@@ -60,6 +60,6 @@
   </link>
   <joint name="base_link_2" type="continuous">
-    <origin xyz="-0.08 0.212 0" rpy="${PI/2} 0 0" />
-    <axis xyz="1 0 0" />
+    <origin xyz="-0.08 0.212 0" rpy="-${PI/2} -${PI/2} 0" />
+    <axis xyz="0 0 1" />
     <parent link="base_link" />
     <child link="wheel_2" />
@@ -69,6 +69,6 @@
   </link>
   <joint name="base_link_3" type="continuous">
-    <origin xyz="0.10934 0.212 0" rpy="${PI/2} 0 0" />
-    <axis xyz="1 0 0" />
+    <origin xyz="0.10934 0.212 0" rpy="-${PI/2} -${PI/2} 0" />
+    <axis xyz="0 0 1" />
     <parent link="base_link" />
     <child link="wheel_3" />
@@ -78,6 +78,6 @@
   </link>
   <joint name="base_link_4" type="continuous">
-    <origin xyz="0.29867 0.212 0" rpy="${PI/2} 0 0" />
-    <axis xyz="1 0 0" />
+    <origin xyz="0.29867 0.212 0" rpy="-${PI/2} -${PI/2} 0" />
+    <axis xyz="0 0 1" />
     <parent link="base_link" />
     <child link="wheel_4" />
@@ -89,5 +89,5 @@
   <joint name="base_link_5" type="continuous">
     <origin xyz="-0.26933 -0.212 0" rpy="${PI/2} 0 0" />
-    <axis xyz="1 0 0" />
+    <axis xyz="0 0 1" />
     <parent link="base_link" />
     <child link="wheel_5" />
@@ -98,5 +98,5 @@
   <joint name="base_link_6" type="continuous">
     <origin xyz="-0.08 -0.212 0" rpy="${PI/2} 0 0" />
-    <axis xyz="1 0 0" />
+    <axis xyz="0 0 1" />
     <parent link="base_link" />
     <child link="wheel_6" />
@@ -107,5 +107,5 @@
   <joint name="base_link_7" type="continuous">
     <origin xyz="0.10934 -0.212 0" rpy="${PI/2} 0 0" />
-    <axis xyz="1 0 0" />
+    <axis xyz="0 0 1" />
     <parent link="base_link" />
     <child link="wheel_7" />
@@ -116,5 +116,5 @@
   <joint name="base_link_8" type="continuous">
     <origin xyz="0.29867 -0.212 0" rpy="${PI/2} 0 0" />
-    <axis xyz="1 0 0" />
+    <axis xyz="0 0 1" />
     <parent link="base_link" />
     <child link="wheel_8" />

Commit message: updated mesh file

File: xacro/bot.xacro (robot description, xacro)
@@ -26,7 +26,7 @@
   <link name="base_link">
   <inertial>
-    <origin xyz="0.089651 0.014045 0.000106459999999999" rpy="0 0 0" />
-    <mass value="4.9511" />
-    <inertia ixx="0.144771700464571" ixy="-0.00641450872692838" ixz="-0.00058647494980373" iyy="0.232027279470688" iyz="-0.000146713403145161" izz="0.369859293842831" />
+    <origin xyz="-0.010263 0.00040996 0.0060706" rpy="0 0 0" />
+    <mass value="18.916" />
+    <inertia ixx="0.23558234792081" ixy="-0.000747515049689842" ixz="-0.0256472781398799" iyy="0.676222174396288" iyz="-0.000297852127122243" izz="0.864544814460253" />
   </inertial>
   <visual>
